File: pcb-modules/max-displays/Modular/DispBrd_DISP/DispBrd_DISP_3+2d/DispBrd_DISP_3+2d.kicad_pcb (KiCad board)
At the start: 2 copper layers, 38.1 x 19.3 mm, 5 parts, among them P10 Disp3+2

Commit message: Max Display panels, modular version FIX: Rear connector rotated 180deg on boards [3+2d], [3+3d], [6x1d] All boards: Silkscreen text on rear oriented correctly; board name added; Format update to KiCAD 6.0.6
Parts:
- moved P10 15.5 mm to (36.8, 29.0), turned to -90 degrees
Routing:
- net /A3: track 4.34 -> 33.0 mm
- net /A4: track 8.98 -> 23.6 mm, vias 0 -> 1
- net /K_SegA: track 30.3 -> 41.6 mm
- net /K_SegB: track 14.2 -> 22.1 mm
- net /A0: track 22.8 -> 16.4 mm
- net /K_SegE: track 33.9 -> 39.4 mm
- net /A2: track 6.88 -> 11.4 mm
- net /A1: track 14.8 -> 10.3 mm
- net /K_SegF: track 34.0 -> 32.1 mm, vias 0 -> 2
- net /K_SegDP: track 26.6 -> 25.5 mm, vias 0 -> 1
- net /K_SegG: track 19.6 -> 18.6 mm
- net /K_SegD: track 34.2 -> 34.7 mm
- net /K_SegC: vias 1 -> 0
Other:
- board text added: "DispBrd [3+2]d GCC 2022-07"
- board text added: "K4 K2 DP F D B"
- board text added: "K5 K3 K1 G E C A"
- board text removed: "A C E G K1 K3 K5"
- board text removed: "B D F dp K2 K4"
