File: pcb-modules/max-displays/Modular/DispBrd_DISP/DispBrd_DISP_3+3d/DispBrd_DISP_3+3d.kicad_pcb (KiCad board)
At the start: 2 copper layers, 46.2 x 19.3 mm, 5 parts, among them P9 Disp3x2

Commit message: Max Display panels, modular version FIX: Rear connector rotated 180deg on boards [3+2d], [3+3d], [6x1d] All boards: Silkscreen text on rear oriented correctly; board name added; Format update to KiCAD 6.0.6
Parts:
- moved P9 15.5 mm to (40.6, 29.0), turned to -90 degrees
Routing:
- net /A5: track 11.7 -> 36.3 mm
- net /A0: track 37.6 -> 15.1 mm
- net /A3: track 4.86 -> 19.0 mm, vias 0 -> 1
- net /A4: track 7.40 -> 20.2 mm
- net /A2: track 15.2 -> 3.81 mm, vias 1 -> 0
- net /A1: track 20.4 -> 12.5 mm
- net /K_SegC: track 26.7 -> 34.5 mm
- net /K_SegA: track 32.7 -> 26.9 mm
- net /K_SegD: track 31.5 -> 26.6 mm, vias 0 -> 1
- net /K_SegG: track 31.0 -> 34.4 mm
- net /K_SegE: track 27.8 -> 30.7 mm, vias 0 -> 1
- net /K_SegB: track 31.4 -> 34.1 mm
- net /K_SegF: track 35.7 -> 33.3 mm, vias 1 -> 0
- net /K_SegDP: track 29.8 -> 27.7 mm, vias 0 -> 1
Other:
- board text added: "DispBrd [3+3]d GCC 2022-07"
- board text added: "K5 K3 K1 G E C A"
- board text added: "K6 K4 K2 dp F D B"
- board text removed: "A C E G K1 K3 K5"
- board text removed: "B D F dp K2 K4 K6"
