File: pcb-modules/max-displays/Modular/DispBrd_DISP/DispBrd_DISP_3d/DispBrd_DISP_3d.kicad_pcb (KiCad board)
At the start: 2 copper layers, 22.4 x 19.3 mm, 4 parts, among them P4 Disp3b

Commit message: Max Display panels, modular version FIX: Rear connector rotated 180deg on boards [3+2d], [3+3d], [6x1d] All boards: Silkscreen text on rear oriented correctly; board name added; Format update to KiCAD 6.0.6
Other:
- board text added: "DispBrd 3d GCC 2022"
- board text added: "K2 dp F D B"
- board text added: "K3 K1 G E C A"
- board text removed: "A C E G K1 K3"
- board text removed: "B D F dp K2"
Changed lines of the file:
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@@
   )
   (gr_rect (start 36.83 13.716) (end 59.182 33.02) (layer "Edge.Cuts") (width 0.05) (fill none))
-  (gr_text "B  D  F  dp K2" (at 46.99 24.13 180) (layer "B.SilkS")
+  (gr_text "K2 dp  F  D  B" (at 46.99 24.13) (layer "B.SilkS")
     (effects (font (size 1.27 1.016) (thickness 0.2032)) (justify mirror))
   )
-  (gr_text "A  C  E  G K1 K3" (at 48.006 18.034 180) (layer "B.SilkS")
+  (gr_text "K3 K1 G  E  C  A" (at 48.006 18.034) (layer "B.SilkS")
     (effects (font (size 1.27 1.016) (thickness 0.2032)) (justify mirror))
   )
+  (gr_text "DispBrd 3d\nGCC 2022" (at 48.006 30.734) (layer "B.SilkS")
+    (effects (font (size 1.397 1.27) (thickness 0.254)) (justify mirror))
+  )
+  (gr_text "DispBrd 3d\nGCC 2022" (at 48.006 30.734) (layer "F.SilkS")
+    (effects (font (size 1.397 1.27) (thickness 0.254)))
+  )
   (segment (start 41.402 18.581) (end 41.949 18.034) (width 0.381) (layer "B.Cu") (net 1))
