File: pcb-modules/max-displays/Modular/DispBrd_DISP/DispBrd_DISP_5d/DispBrd_DISP_5d.kicad_pcb (KiCad board)
At the start: 2 copper layers, 36.6 x 19.3 mm, 4 parts, among them P6 Disp5

Commit message: Max Display panels, modular version FIX: Rear connector rotated 180deg on boards [3+2d], [3+3d], [6x1d] All boards: Silkscreen text on rear oriented correctly; board name added; Format update to KiCAD 6.0.6
Other:
- board text added: "DispBrd 5d GCC 2022-07"
- board text added: "K4 K2 dp F D B"
- board text added: "K5 K3 K1 G E C A"
- board text removed: "A C E G K1 K3 K5"
- board text removed: "B D F dp K2 K4"
Changed lines of the file:
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@@
   )
   (gr_rect (start 50.8 35.814) (end 87.376 55.118) (layer "Edge.Cuts") (width 0.05) (fill none))
-  (gr_text "B  D  F dp K2 K4" (at 68.072 45.974 180) (layer "B.SilkS")
+  (gr_text "K4 K2 dp F  D  B" (at 68.072 46.228) (layer "B.SilkS")
     (effects (font (size 1.27 1.016) (thickness 0.2032)) (justify mirror))
   )
-  (gr_text "A  C  E  G K1 K3 K5" (at 69.342 40.132 180) (layer "B.SilkS")
+  (gr_text "K5 K3 K1 G  E  C  A" (at 69.342 40.132) (layer "B.SilkS")
     (effects (font (size 1.27 1.016) (thickness 0.2032)) (justify mirror))
   )
+  (gr_text "DispBrd 5d\nGCC 2022-07" (at 68.326 52.832) (layer "B.SilkS")
+    (effects (font (size 1.397 1.397) (thickness 0.254)) (justify mirror))
+  )
+  (gr_text "DispBrd 5d\nGCC 2022-07" (at 68.326 52.832) (layer "F.SilkS")
+    (effects (font (size 1.397 1.397) (thickness 0.254)))
+  )
   (segment (start 61.468 41.91) (end 61.468 40.679) (width 0.381) (layer "B.Cu") (net 1))
