File: pcb-modules/max-displays/Modular/DispBrd_DISP/DispBrd_DISP_5dW/DispBrd_DISP_5dW.kicad_pcb (KiCad board)
At the start: 2 copper layers, 47.2 x 14.7 mm, 6 parts, among them P6 Disp5

Commit message: Max Display panels, modular version FIX: Rear connector rotated 180deg on boards [3+2d], [3+3d], [6x1d] All boards: Silkscreen text on rear oriented correctly; board name added; Format update to KiCAD 6.0.6
Other:
- board text added: "DispBrd 5dW GCC 2022-07"
- board text added: "K4 K2 dp F D B"
- board text added: "K5 K3 K1 G E C A"
- board text removed: "A C E G K1 K3 K5"
- board text removed: "B D F dp K2 K4"
Changed lines of the file:
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@@
   )
   (gr_rect (start 35.56 33.02) (end 82.804 47.752) (layer "Edge.Cuts") (width 0.05) (fill none))
-  (gr_text "B  D  F dp K2 K4" (at 58.166 43.18 180) (layer "B.SilkS")
+  (gr_text "K4 K2 dp F  D  B" (at 58.166 43.434) (layer "B.SilkS")
     (effects (font (size 1.27 1.016) (thickness 0.2032)) (justify mirror))
   )
-  (gr_text "A  C  E  G K1 K3 K5" (at 59.69 37.338 180) (layer "B.SilkS")
+  (gr_text "K5 K3 K1 G  E  C  A" (at 59.563 37.465) (layer "B.SilkS")
     (effects (font (size 1.27 1.016) (thickness 0.2032)) (justify mirror))
   )
+  (gr_text "DispBrd 5dW\nGCC 2022-07" (at 74.93 40.386 90) (layer "B.SilkS")
+    (effects (font (size 1.397 1.27) (thickness 0.254)) (justify mirror))
+  )
   (segment (start 51.562 39.116) (end 51.562 37.885) (width 0.381) (layer "B.Cu") (net 1))
