File: pcb-modules/max-displays/Modular/DispBrd_DISP/DispBrd_DISP_6dW/DispBrd_DISP_6dW.kicad_pcb (KiCad board)
At the start: 2 copper layers, 54.4 x 14.7 mm, 6 parts, among them P7 Disp6

Commit message: Max Display panels, modular version FIX: Rear connector rotated 180deg on boards [3+2d], [3+3d], [6x1d] All boards: Silkscreen text on rear oriented correctly; board name added; Format update to KiCAD 6.0.6
Other:
- board text added: "DispBrd 6dW GCC 2022-07"
- board text added: "K5 K3 K1 G E C A"
- board text added: "K6 K4 K2 dp F D B"
- board text removed: "A C E G K1 K3 K5"
- board text removed: "B D F dp K2 K4 K6"
Changed lines of the file:
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@@
   )
   (gr_rect (start 43.18 35.56) (end 97.536 50.292) (layer "Edge.Cuts") (width 0.05) (fill none))
-  (gr_text "A  C  E  G K1 K3 K5" (at 70.612 39.878 180) (layer "B.SilkS")
+  (gr_text "K5 K3 K1 G  E  C  A" (at 70.612 39.878) (layer "B.SilkS")
     (effects (font (size 1.27 1.016) (thickness 0.2032)) (justify mirror))
   )
-  (gr_text "B  D  F dp K2 K4 K6" (at 70.612 45.974 180) (layer "B.SilkS")
+  (gr_text "K6 K4 K2 dp F  D  B" (at 70.612 45.974) (layer "B.SilkS")
     (effects (font (size 1.27 1.016) (thickness 0.2032)) (justify mirror))
   )
+  (gr_text "DispBrd 6dW\nGCC 2022-07" (at 89.408 43.18 90) (layer "B.SilkS")
+    (effects (font (size 1.397 1.27) (thickness 0.254)) (justify mirror))
+  )
   (segment (start 62.738 40.386) (end 65.278 37.846) (width 0.381) (layer "F.Cu") (net 1))
